File: hardware/module-pcb/w41h1-module.kicad_sch (KiCad schematic)
At the start: 31 parts, among them J1 A/C port (2.0 mm, verify), J2 PROG (not fitted), U1 ESP32-C3-WROOM-02, U2 TLV62569DBV, U3 SP3485EN

Commit message: hardware: review fixes for the module PCB, part numbers, fab export
Checked every IC against its datasheet (TLV62569, ESP32-C3-WROOM-02, SP3485):
pinouts, the 0.6 V feedback reference, strapping resistors and the EN delay
match. Two changes came out of it:

- The regulator's output capacitance was above the 47 uF the datasheet allows:
  C3 is 10 uF now.
- The autorouter gave the feedback node a long detour. The regulator is placed
  and pre-routed by hand now: input capacitor, inductor and output capacitor
  next to the part, short switch and feedback nodes.

Also: MPN and LCSC fields on every fitted part, stitch.py keeps vias out of
pads, scripts/fab.sh writes gerbers, drill, BOM, placement file, schematic PDF
and STEP into fab/ after a clean ERC and DRC.

Assisted-by: AI
Parts:
- C1, C2: LCSC (none) -> C45783; MPN (none) -> CL21A226MAQNNNE; Manufacturer (none) -> Samsung
- C3: value 22u 6.3V -> 10u; LCSC (none) -> C15850; MPN (none) -> CL21A106KAYNNNE; Manufacturer (none) -> Samsung
- C4, C7, C8: LCSC (none) -> C14663; MPN (none) -> CC0603KRX7R9BB104; Manufacturer (none) -> Yageo
- C5: LCSC (none) -> C19702; MPN (none) -> CL10A106KP8NNNC; Manufacturer (none) -> Samsung
- C6: LCSC (none) -> C15849; MPN (none) -> CL10A105KB8NNNC; Manufacturer (none) -> Samsung
- D1: value status -> red; LCSC (none) -> C2286; MPN (none) -> KT-0603R; Manufacturer (none) -> Hubei KENTO
- D2: LCSC (none) -> C502564; MPN (none) -> SM712; Manufacturer (none) -> MDD
- J1: LCSC (none) -> C157926; MPN (none) -> S4B-PH-K-S(LF)(SN); Manufacturer (none) -> JST
- L1: LCSC (none) -> C48888311; MPN (none) -> FTC252012S2R2MGCA; Manufacturer (none) -> cjiang
- R1: LCSC (none) -> C25818; MPN (none) -> 0603WAF4533T5E; Manufacturer (none) -> UNI-ROYAL
- R2: LCSC (none) -> C25803; MPN (none) -> 0603WAF1003T5E; Manufacturer (none) -> UNI-ROYAL
- R3, R4, R5, R7, R8, R9: LCSC (none) -> C25804; MPN (none) -> 0603WAF1002T5E; Manufacturer (none) -> UNI-ROYAL
- R6: LCSC (none) -> C21190; MPN (none) -> 0603WAF1001T5E; Manufacturer (none) -> UNI-ROYAL
- U1: LCSC (none) -> C2934560; MPN (none) -> ESP32-C3-WROOM-02-N4; Manufacturer (none) -> Espressif
- U2: LCSC (none) -> C141836; MPN (none) -> TLV62569DBVR; Manufacturer (none) -> Texas Instruments
- U3: LCSC (none) -> C8963; MPN (none) -> SP3485EN-L/TR; Manufacturer (none) -> MaxLinear
Changed lines of the file:
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@@
 			)
 		)
+    (property "MPN" "S4B-PH-K-S(LF)(SN)" (at 30.48 49.53 0)
+      (effects (font (size 1.27 1.27)) (hide yes))
+    )
+    (property "Manufacturer" "JST" (at 30.48 49.53 0)
+      (effects (font (size 1.27 1.27)) (hide yes))
+    )
+    (property "LCSC" "C157926" (at 30.48 49.53 0)
+      (effects (font (size 1.27 1.27)) (hide yes))
+    )
 		(pin "1"
 		)
@@
 			)
 		)
+    (property "MPN" "SM712" (at 59.69 80.01 0)
+      (effects (font (size 1.27 1.27)) (hide yes))
+    )
+    (property "Manufacturer" "MDD" (at 59.69 80.01 0)
+      (effects (font (size 1.27 1.27)) (hide yes))
+    )
+    (property "LCSC" "C502564" (at 59.69 80.01 0)
+      (effects (font (size 1.27 1.27)) (hide yes))
+    )
 		(pin "1"
 		)
@@
 			)
 		)
+    (property "MPN" "CL21A226MAQNNNE" (at 80.01 49.53 0)
+      (effects (font (size 1.27 1.27)) (hide yes))
+    )
+    (property "Manufacturer" "Samsung" (at 80.01 49.53 0)
+      (effects (font (size 1.27 1.27)) (hide yes))
+    )
+    (property "LCSC" "C45783" (at 80.01 49.53 0)
+      (effects (font (size 1.27 1.27)) (hide yes))
+    )
 		(pin "1"
 		)
@@
 			)
 		)
+    (property "MPN" "CC0603KRX7R9BB104" (at 95.25 49.53 0)
+      (effects (font (size 1.27 1.27)) (hide yes))
+    )
+    (property "Manufacturer" "Yageo" (at 95.25 49.53 0)
+      (effects (font (size 1.27 1.27)) (hide yes))
+    )
+    (property "LCSC" "C14663" (at 95.25 49.53 0)
+      (effects (font (size 1.27 1.27)) (hide yes))
+    )
 		(pin "1"
 		)
@@
 			)
 		)
+    (property "MPN" "TLV62569DBVR" (at 124.46 44.45 0)
+      (effects (font (size 1.27 1.27)) (hide yes))
+    )
+    (property "Manufacturer" "Texas Instruments" (at 124.46 44.45 0)
+      (effects (font (size 1.27 1.27)) (hide yes))
+    )
+    (property "LCSC" "C141836" (at 124.46 44.45 0)
+      (effects (font (size 1.27 1.27)) (hide yes))
+    )
 		(pin "1"
 		)
@@
 			)
 		)
+    (property "MPN" "FTC252012S2R2MGCA" (at 154.94 39.37 0)
+      (effects (font (size 1.27 1.27)) (hide yes))
+    )
+    (property "Manufacturer" "cjiang" (at 154.94 39.37 0)
+      (effects (font (size 1.27 1.27)) (hide yes))
+    )
+    (property "LCSC" "C48888311" (at 154.94 39.37 0)
+      (effects (font (size 1.27 1.27)) (hide yes))
+    )
 		(pin "1"
 		)
@@
 			)
 		)
+    (property "MPN" "0603WAF4533T5E" (at 175.26 39.37 0)
+      (effects (font (size 1.27 1.27)) (hide yes))
+    )
+    (property "Manufacturer" "UNI-ROYAL" (at 175.26 39.37 0)
+      (effects (font (size 1.27 1.27)) (hide yes))
+    )
+    (property "LCSC" "C25818" (at 175.26 39.37 0)
+      (effects (font (size 1.27 1.27)) (hide yes))
+    )
 		(pin "1"
 		)
@@
 			)
 		)
+    (property "MPN" "0603WAF1003T5E" (at 175.26 59.69 0)
+      (effects (font (size 1.27 1.27)) (hide yes))
+    )
+    (property "Manufacturer" "UNI-ROYAL" (at 175.26 59.69 0)
+      (effects (font (size 1.27 1.27)) (hide yes))
+    )
+    (property "LCSC" "C25803" (at 175.26 59.69 0)
+      (effects (font (size 1.27 1.27)) (hide yes))
+    )
 		(pin "1"
 		)
@@
 			)
 		)
+    (property "MPN" "CL21A226MAQNNNE" (at 195.58 49.53 0)
+      (effects (font (size 1.27 1.27)) (hide yes))
+    )
+    (property "Manufacturer" "Samsung" (at 195.58 49.53 0)
+      (effects (font (size 1.27 1.27)) (hide yes))
+    )
+    (property "LCSC" "C45783" (at 195.58 49.53 0)
+      (effects (font (size 1.27 1.27)) (hide yes))
+    )
 		(pin "1"
 		)
@@
 			)
 		)
-		(property "Value" "22u 6.3V"
+		(property "Value" "10u"
 			(at 212.09 49.53 0)
 			(show_name no)
@@
 			)
 		)
+    (property "MPN" "CL21A106KAYNNNE" (at 209.55 49.53 0)
+      (effects (font (size 1.27 1.27)) (hide yes))
+    )
+    (property "Manufacturer" "Samsung" (at 209.55 49.53 0)
+      (effects (font (size 1.27 1.27)) (hide yes))
+    )
+    (property "LCSC" "C15850" (at 209.55 49.53 0)
+      (effects (font (size 1.27 1.27)) (hide yes))
+    )
 		(pin "1"
 		)
@@
 			)
 		)
+    (property "MPN" "ESP32-C3-WROOM-02-N4" (at 110.49 129.54 0)
+      (effects (font (size 1.27 1.27)) (hide yes))
+    )
+    (property "Manufacturer" "Espressif" (at 110.49 129.54 0)
+      (effects (font (size 1.27 1.27)) (hide yes))
+    )
+    (property "LCSC" "C2934560" (at 110.49 129.54 0)
+      (effects (font (size 1.27 1.27)) (hide yes))
+    )
 		(pin "1"
 		)
@@
 			)
 		)
+    (property "MPN" "CC0603KRX7R9BB104" (at 149.86 100.33 0)
+      (effects (font (size 1.27 1.27)) (hide yes))
+    )
+    (property "Manufacturer" "Yageo" (at 149.86 100.33 0)
+      (effects (font (size 1.27 1.27)) (hide yes))
+    )
+    (property "LCSC" "C14663" (at 149.86 100.33 0)
+      (effects (font (size 1.27 1.27)) (hide yes))
+    )
 		(pin "1"
 		)
@@
 			)
 		)
+    (property "MPN" "CL10A106KP8NNNC" (at 165.1 100.33 0)
+      (effects (font (size 1.27 1.27)) (hide yes))
+    )
+    (property "Manufacturer" "Samsung" (at 165.1 100.33 0)
+      (effects (font (size 1.27 1.27)) (hide yes))
+    )
+    (property "LCSC" "C19702" (at 165.1 100.33 0)
+      (effects (font (size 1.27 1.27)) (hide yes))
+    )
 		(pin "1"
 		)
@@
 			)
 		)
+    (property "MPN" "0603WAF1002T5E" (at 49.53 105.41 0)
+      (effects (font (size 1.27 1.27)) (hide yes))
+    )
+    (property "Manufacturer" "UNI-ROYAL" (at 49.53 105.41 0)
+      (effects (font (size 1.27 1.27)) (hide yes))
+    )
+    (property "LCSC" "C25804" (at 49.53 105.41 0)
+      (effects (font (size 1.27 1.27)) (hide yes))
+    )
 		(pin "1"
 		)
@@
 			)
 		)
+    (property "MPN" "CL10A105KB8NNNC" (at 49.53 124.46 0)
+      (effects (font (size 1.27 1.27)) (hide yes))
+    )
+    (property "Manufacturer" "Samsung" (at 49.53 124.46 0)
+      (effects (font (size 1.27 1.27)) (hide yes))
+    )
+    (property "LCSC" "C15849" (at 49.53 124.46 0)
+      (effects (font (size 1.27 1.27)) (hide yes))
+    )
 		(pin "1"
 		)
@@
 			)
 		)
+    (property "MPN" "0603WAF1002T5E" (at 35.56 105.41 0)
+      (effects (font (size 1.27 1.27)) (hide yes))
+    )
+    (property "Manufacturer" "UNI-ROYAL" (at 35.56 105.41 0)
+      (effects (font (size 1.27 1.27)) (hide yes))
+    )
+    (property "LCSC" "C25804" (at 35.56 105.41 0)
+      (effects (font (size 1.27 1.27)) (hide yes))
+    )
 		(pin "1"
 		)
@@
 			)
 		)
+    (property "MPN" "0603WAF1002T5E" (at 20.32 105.41 0)
+      (effects (font (size 1.27 1.27)) (hide yes))
+    )
+    (property "Manufacturer" "UNI-ROYAL" (at 20.32 105.41 0)
+      (effects (font (size 1.27 1.27)) (hide yes))
+    )
+    (property "LCSC" "C25804" (at 20.32 105.41 0)
+      (effects (font (size 1.27 1.27)) (hide yes))
+    )
 		(pin "1"
 		)
@@
 			)
 		)
+    (property "MPN" "0603WAF1002T5E" (at 64.77 105.41 0)
+      (effects (font (size 1.27 1.27)) (hide yes))
+    )
+    (property "Manufacturer" "UNI-ROYAL" (at 64.77 105.41 0)
+      (effects (font (size 1.27 1.27)) (hide yes))
+    )
+    (property "LCSC" "C25804" (at 64.77 105.41 0)
+      (effects (font (size 1.27 1.27)) (hide yes))
+    )
 		(pin "1"
 		)
@@
 			)
 		)
+    (property "MPN" "0603WAF1001T5E" (at 20.32 149.86 0)
+      (effects (font (size 1.27 1.27)) (hide yes))
+    )
+    (property "Manufacturer" "UNI-ROYAL" (at 20.32 149.86 0)
+      (effects (font (size 1.27 1.27)) (hide yes))
+    )
+    (property "LCSC" "C21190" (at 20.32 149.86 0)
+      (effects (font (size 1.27 1.27)) (hide yes))
+    )
 		(pin "1"
 		)
@@
 			)
 		)
-		(property "Value" "status"
+		(property "Value" "red"
 			(at 35.56 167.64 0)
 			(show_name no)
@@
 			)
 		)
+    (property "MPN" "KT-0603R" (at 35.56 165.1 0)
+      (effects (font (size 1.27 1.27)) (hide yes))
+    )
+    (property "Manufacturer" "Hubei KENTO" (at 35.56 165.1 0)
+      (effects (font (size 1.27 1.27)) (hide yes))
+    )
+    (property "LCSC" "C2286" (at 35.56 165.1 0)
+      (effects (font (size 1.27 1.27)) (hide yes))
+    )
 		(pin "1"
 		)
@@
 			)
 		)
+    (property "MPN" "SP3485EN-L/TR" (at 214.63 129.54 0)
+      (effects (font (size 1.27 1.27)) (hide yes))
+    )
+    (property "Manufacturer" "MaxLinear" (at 214.63 129.54 0)
+      (effects (font (size 1.27 1.27)) (hide yes))
+    )
+    (property "LCSC" "C8963" (at 214.63 129.54 0)
+      (effects (font (size 1.27 1.27)) (hide yes))
+    )
 		(pin "1"
 		)
@@
 			)
 		)
+    (property "MPN" "CC0603KRX7R9BB104" (at 245.11 100.33 0)
+      (effects (font (size 1.27 1.27)) (hide yes))
+    )
+    (property "Manufacturer" "Yageo" (at 245.11 100.33 0)
+      (effects (font (size 1.27 1.27)) (hide yes))
+    )
+    (property "LCSC" "C14663" (at 245.11 100.33 0)
+      (effects (font (size 1.27 1.27)) (hide yes))
+    )
 		(pin "1"
 		)
@@
 			)
 		)
+    (property "MPN" "0603WAF1002T5E" (at 180.34 149.86 0)
+      (effects (font (size 1.27 1.27)) (hide yes))
+    )
+    (property "Manufacturer" "UNI-ROYAL" (at 180.34 149.86 0)
+      (effects (font (size 1.27 1.27)) (hide yes))
+    )
+    (property "LCSC" "C25804" (at 180.34 149.86 0)
+      (effects (font (size 1.27 1.27)) (hide yes))
+    )
 		(pin "1"
 		)
@@
 			)
 		)
-		(pin "1"
-		)
+    (property "MPN" "0603WAF1002T5E" (at 180.34 110.49 0)
+      (effects (font (size 1.27 1.27)) (hide yes))
+    )
+    (property "Manufacturer" "UNI-ROYAL" (at 180.34 110.49 0)
+      (effects (font (size 1.27 1.27)) (hide yes))
+    )
+    (property "LCSC" "C25804" (at 180.34 110.49 0)
+      (effects (font (size 1.27 1.27)) (hide yes))
+    )
+		(pin "1"
+		)

Commit message: hardware: case for the module PCB, silkscreen labels, final fab outputs
- hardware/module-case: a CadQuery script for a two-part case, 53 x 25 x 11.5 mm.
  Two M2 screws pass through the lid and the board's mounting holes into the base.
  The script checks both parts against the board's STEP model: no overlap.
- Silkscreen labels for the A/C connector pins, the programming pads and the test pads.
- J2 (bare programming pads) is marked as not fitted, so it stays out of the BOM,
  the placement file and the 3D model.
- fab.sh sets the export origin to the board corner and drops unsourced BOM rows.
- READMEs for both, with what was checked and what is still an estimate.

Assisted-by: AI
Parts:
- J2: now not fitted
Changed lines of the file:
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@@
 		(on_board yes)
 		(in_pos_files yes)
-		(dnp no)
+		(dnp yes)
 		(property "Reference" "J2"
 			(at 255.27 157.48 0)

Commit message: hardware: give C1 and C2 the same value so they share one BOM line
Both are the same 22 uF part. Different value text made JLCPCB's importer warn
about two BOM lines matched to one part.

Assisted-by: AI
Parts:
- C1: value 22u 10V -> 22u
- C2: value 22u 6.3V -> 22u
Changed lines of the file:
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@@
 			)
 		)
-		(property "Value" "22u 10V"
+		(property "Value" "22u"
 			(at 82.55 49.53 0)
 			(show_name no)
@@
 			)
 		)
-		(property "Value" "22u 6.3V"
+		(property "Value" "22u"
 			(at 198.12 49.53 0)
 			(show_name no)
